Commit message: new models

File: gym_pepper/assets/models/brick/brick.urdf (robot description, URDF)
Before this commit: robot brick, 1 links, 0 joints
Links:
- link baseLink: mass 0.1 -> None; geometry collision mesh filename=brick.dae scale=1 1 1; visual mesh filename=brick.dae scale=1 1 1

Commit message: brick from Fusion

File: gym_pepper/assets/models/brick/brick.urdf (robot description, URDF)
Before this commit: robot brick, 1 links, 0 joints
Links:
- link baseLink: mass None -> 0.072; geometry collision mesh filename=brick.stl scale=1 1 1; visual mesh filename=brick.stl scale=1 1 1
