Commit message: minor fixes

File: gym_pepper/assets/models/adjustable_table/adjustable_table.urdf (robot description, URDF)
Before this commit: robot adjustable_table, 1 links, 0 joints
Links:
- link baseLink: mass None -> 1.0

Commit message: higher table

File: gym_pepper/assets/models/adjustable_table/adjustable_table.urdf (robot description, URDF)
Before this commit: robot adjustable_table, 1 links, 0 joints
Links:
- link baseLink: geometry collision mesh filename=adjustable_table_tall.dae scale=1 1 1; visual mesh filename=adjustable_table_tall.dae scale=1 1 1
